Commit message: Models and URDF's working

File: urdf/elfin_mount.urdf (robot description, URDF)
Before this commit: robot elfin_mount, 1 links, 0 joints
Links:
- link elfin_mount: geometry collision mesh filename=package://rosi_schunk/mesh/elfin_mount/elfin_mount.STL; visual mesh filename=package://rosi_schunk/mesh/elfin_mount/elfin_mount.STL

File: urdf/schunk_gripper.urdf (robot description, URDF)
Before this commit: robot schunk_gripper, 3 links, 2 joints
Links:
- added link cable_link, mass 0.0012007; collision mesh filename=package://rosi_schunk/mesh/gripper/cable_link.STL; visual mesh filename=package://rosi_schunk/mesh/gripper/cable_link.STL
- added link logo_link, mass 0.00015603; collision mesh filename=package://rosi_schunk/mesh/gripper/logo_link.STL; visual mesh filename=package://rosi_schunk/mesh/gripper/logo_link.STL
- added link sensor_link, mass 0.0033492; collision mesh filename=package://rosi_schunk/mesh/gripper/sensor_link.STL; visual mesh filename=package://rosi_schunk/mesh/gripper/sensor_link.STL
- link schunk_base: mass 0.2178 -> 0.2131
Joints:
- added joint cable_join: type fixed, parent schunk_base, child cable_link, origin xyz=0.0197 0 0.0214 rpy=-1.5708 0 0, axis 0 0 0
- added joint logo_joint: type fixed, parent schunk_base, child logo_link, origin xyz=0 0.0129 0.03915 rpy=-1.5708 0 0, axis 0 0 0
- added joint sensor_joint: type fixed, parent schunk_base, child sensor_link, origin xyz=0.02 -0.0002 0.0696 rpy=1.5708 0 -1.5708, axis 0 0 0
- joint finge2_joint: axis 0 0 0 -> 0 -1 0
- joint finger1_joint: axis 0 0 0 -> 0 0 1
