Commit message: Updated limit direction

File: urdf/schunk_gripper.urdf (robot description, URDF)
Before this commit: robot schunk_gripper, 6 links, 5 joints
Joints:
- removed joint finge2_joint
- added joint finger2_joint: type prismatic, parent schunk_base, child finger2_link, origin xyz=0.014 0.004 0.08105 rpy=3.1416 0 -1.5708, axis 0 -1 0, limit lower=0 upper=0.006 effort=72.5 velocity=0.03, mimic joint=finger1_joint multiplier=-1 offset=0
- joint finger1_joint: limit lower=0 upper=0.006 effort=72.5 velocity=0.03 -> lower=-0.006 upper=0 effort=72.5 velocity=0.03

Commit message: Fixed typo and added transmissions

File: urdf/schunk_gripper.urdf (robot description, URDF)
Before this commit: robot schunk_gripper, 6 links, 5 joints
Joints:
- removed joint cable_join
- added joint cable_joint: type fixed, parent schunk_base, child cable_link, origin xyz=0.0197 0 0.0214 rpy=-1.5708 0 0, axis 0 0 0

Commit message: mimic removed

File: urdf/schunk_gripper.urdf (robot description, URDF)
Before this commit: robot schunk_gripper, 6 links, 5 joints
Joints:
- joint finger2_joint: mimic joint=finger1_joint multiplier=-1 offset=0 -> (none)
